File: kicad/WLAN.kicad_sch (KiCad schematic)
At the start: 1 part

Commit message: finished bluetooth schematic apart from anteantenna-design, WiFi design started
Parts:
- removed U?: ESP8266EX, Package_DFN_QFN:QFN-32-1EP_5x5mm_P0.5mm_EP3.45x3.45mm, symbol MCU_Espressif:ESP8266EX
Changed lines of the file:
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@@
 	(generator_version "8.0")
 	(paper "A4")
-	(symbol
-		(lib_id "MCU_Espressif:ESP8266EX")
-		(at 82.55 95.25 0)
-		(unit 1)
-		(exclude_from_sim no)
-		(in_bom yes)
-		(on_board yes)
-		(dnp no)
-		(fields_autoplaced yes)
-		(property "Reference" "U?"
-			(at 84.7441 123.44 0)
-			(effects
-				(font
-					(size 1.27 1.27)
-				)
-				(justify left)
-			)
-		)
-		(property "Value" "ESP8266EX"
-			(at 84.7441 125.98 0)
-			(effects
-				(font
-					(size 1.27 1.27)
-				)
-				(justify left)
-			)
-		)
-		(property "Footprint" "Package_DFN_QFN:QFN-32-1EP_5x5mm_P0.5mm_EP3.45x3.45mm"
-			(at 82.55 128.27 0)
-			(effects
-				(font
-					(size 1.27 1.27)
-				)
-				(hide yes)
-			)
-		)
-		(property "Datasheet" "http://espressif.com/sites/default/files/documentation/0a-esp8266ex_datasheet_en.pdf"
-			(at 85.09 128.27 0)
-			(effects
-				(font
-					(size 1.27 1.27)
-				)
-				(hide yes)
-			)
-		)
-		(property "Description" "Highly integrated Wi-Fi SoC, QFN-32"
-			(at 82.55 95.25 0)
-			(effects
-				(font
-					(size 1.27 1.27)
-				)
-				(hide yes)
-			)
-		)
-		(pin "26"
-		)
-		(pin "25"
-		)
-		(pin "3"
-		)
-		(pin "4"
-		)
-		(pin "23"
-		)
-		(pin "8"
-		)
-		(pin "7"
-		)
-		(pin "30"
-		)
-		(pin "32"
-		)
-		(pin "21"
-		)
-		(pin "10"
-		)
-		(pin "28"
-		)
-		(pin "13"
-		)
-		(pin "27"
-		)
-		(pin "5"
-		)
-		(pin "18"
-		)
-		(pin "6"
-		)
-		(pin "29"
-		)
-		(pin "9"
-		)
-		(pin "17"
-		)
-		(pin "19"
-		)
-		(pin "22"
-		)
-		(pin "2"
-		)
-		(pin "15"
-		)
-		(pin "31"
-		)
-		(pin "24"
-		)
-		(pin "11"
-		)
-		(pin "14"
-		)
-		(pin "12"
-		)
-		(pin "33"
-		)
-		(pin "1"
-		)
-		(pin "16"
-		)
-		(pin "20"
-		)
-		(instances
-			(project ""
-				(path "/601a88ea-2da7-4ec4-b637-f587eb4ba821/e37a04e5-c2cd-4971-ba15-bb62af991442"
-					(reference "U?")
-					(unit 1)
-				)
-			)
-		)
-	)
 )
